File: PCB/JAARK_PCB_MOTOR/JAARK_PCB_MOTOR.kicad_sch (KiCad schematic)
At the start: 51 parts, among them IC1 TPS564242DRLR, IC2 PJA3404_R1_00001, IC3 PJA3404_R1_00001, IC4 HIP4080AIBZT, IC5 PJA3404_R1_00001, IC6 PJA3404_R1_00001, IC7 PJA3404_R1_00001, IC8 PJA3404_R1_00001, J1 Battery Terminal, J2 Morpho_x2_SSW-119-01-T-D, Q1 SSM3J334RLF, Q2 SSM3J334RLF, Q3 FMMT619TA, Q4 FMMT619TA, Q5 FMMT619TA, Q6 SSM3J334RLF, Q7 FMMT619TA

Commit message: Better motor drivers, fixed capacitor in voltage regulation.
Parts:
- removed C8: 22uF, JAARK_lib:CAPC2012X95N, symbol JAARK_lib:CL21B104KBCNNNC
- added C10, C9: 100uF, JAARK_lib:CAPC3216X180N, symbol Device:C_Small
- added C11, C12, C14: 33uF, JAARK_lib:CAPC3216X180N, symbol Device:C_Small
- added C13, C15: 0.1uF, C0805, symbol Device:C_Small
- added D2, D3: S2JTR, Diode_SMD:D_SMB, symbol Diode:S2JTR
- added D4: 15V, Diode_SMD:D_SOD-923, symbol Diode:ESD9B3.3ST5G
- added IC10, IC9: DRV8231DDAR, SOIC127P600X170-9N, symbol JAARK_lib:DRV8231DDAR
- added J5, J6: ~, JAARK_lib:1984617, symbol SSys_Parts:1984617
- added R10, R11: 0.2R, symbol Device:R_Small_US
- added R5, R6, R8, R9: 20kR, RESC2012X50N, symbol Device:R_Small_US
- C6: value 33uF -> 220pF; footprint JAARK_lib:CAPC3216X180N -> CAPC2012X75N; Arrow Part Number C3216X5R1E336M160AC -> CL21C221JBANNNC; Arrow Price/Stock https://www.arrow.com/en/products/c3216x5r1e336m160ac/tdk -> https://www.arrow.com/en/products/cl21c221jbannnc/samsung-e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; Height 1.8 -> 0.75; Manufacturer_Name TDK -> SAMSUNG; Manufacturer_Part_Number C3216X5R1E336M160AC -> CL21C221JBANNNC; Mouser Part Number 810-C3216X5R1E336M -> 187-CL21C221JBANNNC; Mouser Price/Stock https://www.mouser.co.uk/ProductDetail/TDK/C3216X5R1E336M16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 -> https://www.mouser.co.uk/ProductDetail/Samsung-Electro-Mech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
- D10, D11, D8, D9, IC2, IC3, IC4, IC5, IC6, IC7, IC8, J3, J4, Q2, Q3, Q4, Q5, Q6, Q7, R14, R15, R16, R17, R18, R19, R20, R21, R22, R7: now left out of the parts list
- F1: value 5A -> 4A
Connections:
- net +12V: now also IC4.16 (VDD), IC4.2 (HEN), C12.2, C13.1, C14.2, C15.1, D2.2 (A), D3.2 (A), D4.2 (A2), IC10.5 (VM), IC9.5 (VM)
- net GND: now also IC4.14 (ALS), IC4.17 (BLS), IC4.3 (DIS), IC4.4 (VSS), C12.1, C13.2, C14.1, C15.2, D4.1 (A1), IC10.1 (GND), IC10.9 (EP), IC9.1 (GND), IC9.9 (EP), R10.2, R11.2, R5.2, R6.2, R8.2; no longer C7.2
- net at IC4.19 (BHS), IC5.2 (S), IC6.3 (D)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: now also C9.1
- net at IC4.12 (AHS), IC7.2 (S), IC8.3 (D)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: now also C10.1
- net at IC4.1 (BHB): now also C9.2, D3.1 (K)
- net at IC4.10 (AHB): now also C10.2, D2.1 (K)
- net at IC4.5 (OUT): now also C11.2, R9.2
- net IN1_MTR: now reaches IC4.6 (IN+)
- net IN1_MTR: now also C11.1, R9.1
- net IN2_MTR: now reaches IC4.7 (IN-)
- net at IC4.8 (HDEL): now also R6.1
- net at IC4.9 (LDEL): now also R8.1
- new net: IC10.6 (OUT1), J6.2
- new net: IC10.7 (ISEN), R11.1
- new net: IC10.8 (OUT2), J6.1
- new net: IC9.7 (ISEN), R10.1
- new net: C7.2, R5.1
- new net: IC9.6 (OUT1), J5.2
- new net: IC9.8 (OUT2), J5.1
- new net +3V3: IC10.4 (VREF), IC9.4 (VREF)
- new net IN1: IC10.2 (IN2), IC9.2 (IN2)
- new net IN2: IC10.3 (IN1), IC9.3 (IN1)
Other:
- note added: "I(OUTX) <= 1.6 Amps"
- note added: "Motor Driver 1"
- note added: "Motor Driver 2"
- note removed: "H-Bridge (Motor Controller)"
- moved on the sheet: C1, C2, C3, C4, C5, C6, C7, D1, F1, IC1, IC4, IC5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

Commit message: PCB Motor V1 finished.
Parts:
- removed D1: D_Zener, symbol Device:D_Zener
- removed F1: 4A, symbol Device:Fuse
- removed J2: Morpho_x2_SSW-119-01-T-D, footprint_library:STM_Nucleo_Morpho_x2_Footprint, symbol sym_library:Morpho_x2_SSW-119-01-T-D
- removed V1: 12, symbol Simulation_SPICE:VDC
- added J2: Morpho_x2_SSW-119-01-T-D, JAARK_lib:STM_Nucleo_Morpho_x2_Footprint, symbol JAARK_lib:Morpho_x2_SSW-119-01-T-D
- added U1: 4A, JAARK_lib:3586TR, symbol JAARK_lib:Fuse
- C13, C15, C3: footprint C0805 -> JAARK_lib:C0805
- C6: footprint CAPC2012X75N -> JAARK_lib:CAPC2012X75N
- C7: footprint (none) -> JAARK_lib:CAPAE660X800N; symbol Device:C_Polarized_Small -> JAARK_lib:UWT1V101MCL1GS; Arrow Part Number (none) -> UWT1V101MCL1GS; Arrow Price/Stock (none) -> https://www.arrow.com/en/products/uwt1v101mcl1gs/nichicon?u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; Height (none) -> 8; Manufacturer_Name (none) -> Nichicon; Manufacturer_Part_Number (none) -> UWT1V101MCL1GS; Mouser Part Number (none) -> 647-UWT1V101MCL1S; Mouser Price/Stock (none) -> https://www.mouser.co.uk/ProductDetail/Nichicon/UWT1V101MCL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
- D4: footprint Diode_SMD:D_SOD-923 -> JAARK_lib:SODFL3616X135N; Height (none) -> 1.35; Manufacturer_Name (none) -> MCC; Manufacturer_Part_Number (none) -> SMF12CA
- IC10, IC9: footprint SOIC127P600X170-9N -> JAARK_lib:SOIC127P600X170-9N
- L1: footprint INDPM4141X200N -> JAARK_lib:INDPM4141X200N
- Q1: footprint 2SC2712GRLF -> JAARK_lib:2SC2712GRLF; Spice_Node_Sequence 3 1 2 2 -> (none)
- R1: footprint RESC2012X65N -> JAARK_lib:RESC2012X65N
- R10: footprint (none) -> JAARK_lib:RESC2013X65N; symbol Device:R_Small_US -> JAARK_lib:R_Small_US; Manufacturer_Name (none) -> Susumu; Manufacturer_Part_Number (none) -> RL1220S-R20-F; Mouser Part Number (none) -> 754-RL1220S-R20-F; Mouser Price/Stock (none) -> https://www.mouser.co.uk/ProductDetail/Susumu/RL1220S-R20-F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
- R11: footprint (none) -> JAARK_lib:RESC2013X65N; Manufacturer_Name (none) -> Susumu; Manufacturer_Part_Number (none) -> RL1220S-R20-F; Mouser Part Number (none) -> 754-RL1220S-R20-F; Mouser Price/Stock (none) -> https://www.mouser.co.uk/ProductDetail/Susumu/RL1220S-R20-F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
- R2: footprint RESC2012X60N -> JAARK_lib:RESC2012X60N
- R3, R5: footprint RESC2012X50N -> JAARK_lib:RESC2012X50N
Connections:
- net +3V3: now also J2.A16 (+3V3)
- net +5V: now also J2.A6 (E5V)
- net GND: now also J2.A19 (GND), J2.A20 (GND), J2.A22 (GND), J2.A8 (GND), J2.B9 (GND)
- net IN1: now also J2.A38 (PC0); no longer IC10.2 (IN2)
- net IN2: now also J2.A36 (PC1); no longer IC10.3 (IN1)
- net at J1.2: now also U1.1
- net at Q1.3 (D): now also U1.2
- new net IN3: IC10.2 (IN2), J2.B37 (PA3)
- new net IN4: IC10.3 (IN1), J2.B35 (PA2)
Other:
- moved on the sheet: D4, V2, V3
